File: KiCAD/DC-DC-only/DC-DC-only.sch (KiCad schematic (older format))
At the start: 20 parts, among them J1 V_In, J2 GND, J3 V_Out, J4 GND, U1 TPS54331D

Commit message: Add new 3d footprint for SLO0630H
Parts:
- added H1, H2, H3, H4: MountingHole, MeineBibpretty:EigenesMountingHole_2.7mm_M2.5, symbol Mechanical:MountingHole
- added LO1: Logo, MeineBibpretty:Binary_6_v0.1, symbol Mechanical:MountingHole
Changed lines of the file:
@@
 Wire Wire Line
 	8450 4300 8550 4300
+$Comp
+L Mechanical:MountingHole H1
+U 1 1 60061C46
+P 2250 6250
+F 0 "H1" H 2350 6296 50  0000 L CNN
+F 1 "MountingHole" H 2350 6205 50  0000 L CNN
+F 2 "MeineBibpretty:EigenesMountingHole_2.7mm_M2.5" H 2250 6250 50  0001 C CNN
+F 3 "~" H 2250 6250 50  0001 C CNN
+	1    2250 6250
+	1    0    0    -1
+$EndComp
+$Comp
+L Mechanical:MountingHole H2
+U 1 1 6006263D
+P 2250 6450
+F 0 "H2" H 2350 6496 50  0000 L CNN
+F 1 "MountingHole" H 2350 6405 50  0000 L CNN
+F 2 "MeineBibpretty:EigenesMountingHole_2.7mm_M2.5" H 2250 6450 50  0001 C CNN
+F 3 "~" H 2250 6450 50  0001 C CNN
+	1    2250 6450
+	1    0    0    -1
+$EndComp
+$Comp
+L Mechanical:MountingHole H3
+U 1 1 60062968
+P 2250 6650
+F 0 "H3" H 2350 6696 50  0000 L CNN
+F 1 "MountingHole" H 2350 6605 50  0000 L CNN
+F 2 "MeineBibpretty:EigenesMountingHole_2.7mm_M2.5" H 2250 6650 50  0001 C CNN
+F 3 "~" H 2250 6650 50  0001 C CNN
+	1    2250 6650
+	1    0    0    -1
+$EndComp
+$Comp
+L Mechanical:MountingHole H4
+U 1 1 60062D80
+P 2250 6850
+F 0 "H4" H 2350 6896 50  0000 L CNN
+F 1 "MountingHole" H 2350 6805 50  0000 L CNN
+F 2 "MeineBibpretty:EigenesMountingHole_2.7mm_M2.5" H 2250 6850 50  0001 C CNN
+F 3 "~" H 2250 6850 50  0001 C CNN
+	1    2250 6850
+	1    0    0    -1
+$EndComp
+$Comp
+L Mechanical:MountingHole LO1
+U 1 1 600638EF
+P 3150 6250
+F 0 "LO1" H 3250 6296 50  0000 L CNN
+F 1 "Logo" H 3250 6205 50  0000 L CNN
+F 2 "MeineBibpretty:Binary_6_v0.1" H 3150 6250 50  0001 C CNN
+F 3 "~" H 3150 6250 50  0001 C CNN
+	1    3150 6250
+	1    0    0    -1
+$EndComp
 $EndSCHEMATC

Commit message: Create v0.1 of DC-DC-only PCB and export gerber files
Parts:
- removed H2, H4: MountingHole, MeineBibpretty:EigenesMountingHole_2.7mm_M2.5, symbol Mechanical:MountingHole
- added D2: SS14, Diode_SMD:D_SMA, symbol MeineBibli:SS14
Connections:
- net GND: now also C8.2, C9.2, D1.2 (A), U1.7 (GND)
- net at C8.1, C9.1, L1.2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: now also D2.2 (A); no longer J3.1 (Pin_1)
- new net: D2.1 (K), J3.1 (Pin_1)
Changed lines of the file:
@@
 	6700 2850 7100 2850
 Wire Wire Line
-	6000 3550 6700 3550
+	6000 3550 6350 3550
 Wire Wire Line
 	6700 3550 6700 3350
@@
 Wire Wire Line
 	7950 3350 7950 2850
-Connection ~ 7950 2850
-Wire Wire Line
-	7950 2850 8550 2850
 Connection ~ 7950 3750
 Wire Wire Line
@@
 $EndComp
 $Comp
-L Mechanical:MountingHole H2
-U 1 1 6006263D
-P 2250 6450
-F 0 "H2" H 2350 6496 50  0000 L CNN
-F 1 "MountingHole" H 2350 6405 50  0000 L CNN
-F 2 "MeineBibpretty:EigenesMountingHole_2.7mm_M2.5" H 2250 6450 50  0001 C CNN
-F 3 "~" H 2250 6450 50  0001 C CNN
-	1    2250 6450
-	1    0    0    -1
-$EndComp
-$Comp
 L Mechanical:MountingHole H3
 U 1 1 60062968
@@
 F 3 "~" H 2250 6650 50  0001 C CNN
 	1    2250 6650
-	1    0    0    -1
-$EndComp
-$Comp
-L Mechanical:MountingHole H4
-U 1 1 60062D80
-P 2250 6850
-F 0 "H4" H 2350 6896 50  0000 L CNN
-F 1 "MountingHole" H 2350 6805 50  0000 L CNN
-F 2 "MeineBibpretty:EigenesMountingHole_2.7mm_M2.5" H 2250 6850 50  0001 C CNN
-F 3 "~" H 2250 6850 50  0001 C CNN
-	1    2250 6850
 	1    0    0    -1
 $EndComp
@@
 	1    0    0    -1
 $EndComp
+$Comp
+L power:GND #PWR0107
+U 1 1 6008808E
+P 6350 3600
+F 0 "#PWR0107" H 6350 3350 50  0001 C CNN
+F 1 "GND" H 6350 3750 50  0000 C CNN
+F 2 "" H 6350 3600 50  0001 C CNN
+F 3 "" H 6350 3600 50  0001 C CNN
+	1    6350 3600
+	1    0    0    -1
+$EndComp
+Wire Wire Line
+	6350 3600 6350 3550
+Connection ~ 6350 3550
+Wire Wire Line
+	6350 3550 6700 3550
+$Comp
+L MeineBibli:SS14 D2
+U 1 1 60089C96
+P 8250 2850
+F 0 "D2" H 8200 2750 50  0000 L CNN
+F 1 "SS14" H 8150 2950 50  0000 L CNN
+F 2 "Diode_SMD:D_SMA" H 8250 2675 50  0001 C CNN
+F 3 "https://datasheet.lcsc.com/szlcsc/1903051003_MDD-Jiangsu-Yutai-Elec-SS14_C2480.pdf" H 8250 2850 50  0001 C CNN
+F 4 "C2480" V 8341 2930 50  0001 L CNN "LCSC"
+	1    8250 2850
+	-1   0    0    1
+$EndComp
+Wire Wire Line
+	7950 2850 8100 2850
+Connection ~ 7950 2850
+Wire Wire Line
+	8400 2850 8550 2850
 $EndSCHEMATC
