File: KiCAD/DC-DC-only/DC-DC-only.kicad_pcb (KiCad board)
At the start: 2 copper layers, 20 parts, among them J1 V_In, J2 GND, J3 V_Out, J4 GND, U1 TPS54331D

Commit message: Create v0.1 of DC-DC-only PCB and export gerber files
Parts:
- added D2: SS14, Diode_SMD:D_SMA, F.Cu at (138.5, 86.9)
- added H1: MountingHole, MeineBibpretty:EigenesMountingHole_2.7mm_M2.5, F.Cu at (112.0, 82.6)
- added H3: MountingHole, MeineBibpretty:EigenesMountingHole_2.7mm_M2.5, F.Cu at (138.0, 97.6)
- added LO1: Logo, MeineBibpretty:Binary_6_v0.1, F.Cu at (125.0, 82.6)
- moved C3 46.1 mm to (116.5, 93.1), turned to 90 degrees
- moved R7 44.6 mm to (130.2, 98.3), turned to 180 degrees
- moved C5 44.2 mm to (116.5, 96.3), turned to 270 degrees
- moved J2 40.1 mm to (145.6, 99.1), turned to 270 degrees
- moved J4 38.7 mm to (105.0, 99.0), turned to 90 degrees
- moved R5 35.4 mm to (129.4, 96.0), turned to 270 degrees
- moved C1 35.2 mm to (111.9, 95.5), turned to 270 degrees
- moved J1 34.2 mm to (105.0, 81.2), turned to 90 degrees
- moved C7 33.7 mm to (127.8, 96.0), turned to 270 degrees
- moved C9 32.8 mm to (138.7, 91.1), turned to 270 degrees
- moved D1 32.1 mm to (123.4, 89.7), turned to 180 degrees
- moved L1 29.8 mm to (130.9, 89.7)
- moved C4 29.4 mm to (126.1, 93.0), turned to 270 degrees
- moved C8 28.6 mm to (136.1, 91.1), turned to 270 degrees
- moved U1 27.0 mm to (121.0, 94.5)
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Connections:
- C8 pad 2: Net-(C8-Pad2) -> GND
- C9 pad 2: Net-(C8-Pad2) -> GND
- D1 pad 2: Net-(C8-Pad2) -> GND
- J3 pad 1: Net-(C8-Pad1) -> Net-(D2-Pad1)
- U1 pad 7: Net-(C8-Pad2) -> GND
Routing:
- net GND: track 0.00 -> 68.3 mm
- net Net-(C1-Pad1): track 0.00 -> 24.5 mm
- net Net-(C8-Pad1): track 0.00 -> 16.2 mm
- net Net-(R5-Pad2): track 0.00 -> 13.1 mm, vias 0 -> 2
- net Net-(C4-Pad2): track 0.00 -> 12.7 mm, vias 0 -> 2
- net Net-(D2-Pad1): track 0.00 -> 9.91 mm
- net Net-(C4-Pad1): track 0.00 -> 7.96 mm
- net Net-(C6-Pad1): track 0.00 -> 4.30 mm
- net Net-(C5-Pad1): track 0.00 -> 2.48 mm
- net Net-(C6-Pad2): track 0.00 -> 1.52 mm
- net Net-(R6-Pad2): track 0.00 -> 1.47 mm
- added copper zone on B.Cu, net GND
- added copper zone on F.Cu, net GND
Other:
- board outline added: 44.6 x 21.8 mm
- net class Power added: clearance 0.2, trace_width 0.5, via_dia 0.8, via_drill 0.4
- board text added: "TPS54331 DC-DC converter Vin = 12 - 28 V Vout = 5 V after diode v0.1 - Chrismettal 2020"

Commit message: Port DC-DC-only to KiCAD 5.99, remove rescue libs, order CP2102 USB gerbers
Connections:
- U1 pad 3: Net-(U1-Pad3) -> unconnected-(U1-Pad3)
Other:
- net class Default removed
- net class Power removed
