File: KiCAD/ESP-Hiro/ESP-Hiro.sch (KiCad schematic (older format))
At the start: 69 parts, among them J1 Conn_Q1, J2 Conn_Q2, J3 Conn_Q3, J4 Conn_Q4, J5 Conn_Q5, J6 Conn_ADC, Q1 AO3400A, Q2 AO3400A, Q3 AO3400A, Q4 AO3400A, Q5 AO3400A, U1 DHT22/DS18B20 header, U2 ESP-12E, U3 TPS54331D, U4 TLV75533PDBVR

Commit message: Dump all new components to PCB
Parts:
- gave numbers to parts that had none: 13
Changed lines of the file:
@@
 $EndComp
 $Comp
-L Connector:USB_C_Receptacle_USB2.0 J?
+L Connector:USB_C_Receptacle_USB2.0 J7
 U 1 1 60188C1E
 P 1500 5750
-F 0 "J?" H 1500 6500 50  0000 C CNN
+F 0 "J7" H 1500 6500 50  0000 C CNN
 F 1 "Korean Hroparts TYPE-C-31-M-12" V 1000 5750 50  0000 C CNN
 F 2 "Connector_USB:USB_C_Receptacle_HRO_TYPE-C-31-M-12" H 1650 5750 50  0001 C CNN
@@
 $EndComp
 $Comp
-L Interface_USB:CP2102N-A01-GQFN28 U?
+L Interface_USB:CP2102N-A01-GQFN28 U5
 U 1 1 6023C75C
 P 4300 5850
-F 0 "U?" H 4450 4550 50  0000 C CNN
+F 0 "U5" H 4450 4550 50  0000 C CNN
 F 1 "CP2102N-A01-GQFN28" H 4850 4450 50  0000 C CNN
 F 2 "Package_DFN_QFN:QFN-28-1EP_5x5mm_P0.5mm_EP3.35x3.35mm" H 4750 4650 50  0001 L CNN
@@
 $EndComp
 $Comp
-L power:GND #PWR?
+L power:GND #PWR0101
 U 1 1 6023E253
 P 1200 6850
-F 0 "#PWR?" H 1200 6600 50  0001 C CNN
+F 0 "#PWR0101" H 1200 6600 50  0001 C CNN
 F 1 "GND" H 1205 6677 50  0000 C CNN
 F 2 "" H 1200 6850 50  0001 C CNN
@@
 	2200 5850 2700 5850
 $Comp
-L power:VBUS #PWR?
+L power:VBUS #PWR0102
 U 1 1 602A343F
 P 2800 4650
-F 0 "#PWR?" H 2800 4500 50  0001 C CNN
+F 0 "#PWR0102" H 2800 4500 50  0001 C CNN
 F 1 "VBUS" H 2815 4823 50  0000 C CNN
 F 2 "" H 2800 4650 50  0001 C CNN
@@
 P 4300 4200
 AR Path="/601D55C5/602B1B9F" Ref="#PWR?"  Part="1"
-AR Path="/602B1B9F" Ref="#PWR?"  Part="1"
-F 0 "#PWR?" H 4300 4050 50  0001 C CNN
+AR Path="/602B1B9F" Ref="#PWR0103"  Part="1"
+F 0 "#PWR0103" H 4300 4050 50  0001 C CNN
 F 1 "+3.3V" H 4300 4350 50  0000 C CNN
 F 2 "" H 4300 4200 50  0001 C CNN
@@
 Connection ~ 4300 4450
 $Comp
-L power:GND #PWR?
+L power:GND #PWR0104
 U 1 1 602DB25B
 P 4300 7250
-F 0 "#PWR?" H 4300 7000 50  0001 C CNN
+F 0 "#PWR0104" H 4300 7000 50  0001 C CNN
 F 1 "GND" H 4305 7077 50  0000 C CNN
 F 2 "" H 4300 7250 50  0001 C CNN
@@
 P 3550 4550
 AR Path="/601D55C5/602E9F87" Ref="C?"  Part="1"
-AR Path="/602E9F87" Ref="C?"  Part="1"
-F 0 "C?" H 3400 4450 50  0000 L CNN
+AR Path="/602E9F87" Ref="C17"  Part="1"
+F 0 "C17" H 3400 4450 50  0000 L CNN
 F 1 "100nF" H 3300 4650 50  0000 L CNN
 F 2 "Capacitor_SMD:C_0603_1608Metric" H 3550 4550 50  0001 C CNN
@@
 P 3150 6650
 AR Path="/601D55C5/602EDDC8" Ref="C?"  Part="1"
-AR Path="/602EDDC8" Ref="C?"  Part="1"
-F 0 "C?" H 3000 6550 50  0000 L CNN
+AR Path="/602EDDC8" Ref="C15"  Part="1"
+F 0 "C15" H 3000 6550 50  0000 L CNN
 F 1 "100nF" H 2900 6750 50  0000 L CNN
 F 2 "Capacitor_SMD:C_0603_1608Metric" H 3150 6650 50  0001 C CNN
@@
 $EndComp
 $Comp
-L power:GND #PWR?
+L power:GND #PWR0105
 U 1 1 603027BC
 P 3550 4800
-F 0 "#PWR?" H 3550 4550 50  0001 C CNN
+F 0 "#PWR0105" H 3550 4550 50  0001 C CNN
 F 1 "GND" H 3555 4627 50  0000 C CNN
 F 2 "" H 3550 4800 50  0001 C CNN
@@
 	3150 6500 3150 6400
 $Comp
-L power:GND #PWR?
+L power:GND #PWR0106
 U 1 1 6037461C
 P 3150 7000
-F 0 "#PWR?" H 3150 6750 50  0001 C CNN
+F 0 "#PWR0106" H 3150 6750 50  0001 C CNN
 F 1 "GND" H 3155 6827 50  0000 C CNN
 F 2 "" H 3150 7000 50  0001 C CNN
@@
 	3150 7000 3150 6900
 $Comp
-L Device:R R?
+L Device:R R26
 U 1 1 60392901
 P 5050 5050
-F 0 "R?" V 5100 5200 50  0000 C CNN
+F 0 "R26" V 5100 5200 50  0000 C CNN
 F 1 "470R" V 5050 5050 50  0000 C CNN
 F 2 "Resistor_SMD:R_0603_1608Metric" V 4980 5050 50  0001 C CNN
@@
 P 6000 4850
 AR Path="/601D55C5/603D2CD6" Ref="R?"  Part="1"
-AR Path="/603D2CD6" Ref="R?"  Part="1"
-F 0 "R?" V 6100 4850 50  0000 C CNN
+AR Path="/603D2CD6" Ref="R27"  Part="1"
+F 0 "R27" V 6100 4850 50  0000 C CNN
 F 1 "12k" V 6000 4850 50  0000 C CNN
 F 2 "Resistor_SMD:R_0603_1608Metric" V 5930 4850 50  0001 C CNN
@@
 P 6000 5450
 AR Path="/601D55C5/603D5003" Ref="R?"  Part="1"
-AR Path="/603D5003" Ref="R?"  Part="1"
-F 0 "R?" V 6100 5450 50  0000 C CNN
+AR Path="/603D5003" Ref="R28"  Part="1"
+F 0 "R28" V 6100 5450 50  0000 C CNN
 F 1 "12k" V 6000 5450 50  0000 C CNN
 F 2 "Resistor_SMD:R_0603_1608Metric" V 5930 5450 50  0001 C CNN
@@
 $EndComp
 $Comp
-L MeineBibli:S8050_correctpins Q?
+L MeineBibli:S8050_correctpins Q6
 U 1 1 603D6656
 P 6450 4850
-F 0 "Q?" H 6641 4896 50  0000 L CNN
+F 0 "Q6" H 6641 4896 50  0000 L CNN
 F 1 "S8050_correctpins" H 6641 4805 50  0000 L CNN
 F 2 "Package_TO_SOT_SMD:SOT-23" H 6650 4775 50  0001 L CIN
@@
 	6150 4850 6250 4850
 $Comp
-L MeineBibli:S8050_correctpins Q?
+L MeineBibli:S8050_correctpins Q7
 U 1 1 603E79DA
 P 6450 5450
-F 0 "Q?" H 6641 5404 50  0000 L CNN
+F 0 "Q7" H 6641 5404 50  0000 L CNN
 F 1 "S8050_correctpins" H 6641 5495 50  0000 L CNN
 F 2 "Package_TO_SOT_SMD:SOT-23" H 6650 5375 50  0001 L CIN
@@
 	4900 5450 5750 5450
 $Comp
-L MeineBibli:SS14 D?
+L MeineBibli:SS14 D2
 U 1 1 6057A53A
 P 3150 4900
-F 0 "D?" V 3000 4900 50  0000 L CNN
+F 0 "D2" V 3000 4900 50  0000 L CNN
 F 1 "SS14" V 3250 4900 50  0000 L CNN
 F 2 "Diode_SMD:D_SMA" H 3150 4725 50  0001 C CNN
@@
 P 3150 4650
 AR Path="/601D55C5/60630B5B" Ref="#PWR?"  Part="1"
-AR Path="/60630B5B" Ref="#PWR?"  Part="1"
-F 0 "#PWR?" H 3150 4500 50  0001 C CNN
+AR Path="/60630B5B" Ref="#PWR0107"  Part="1"
+F 0 "#PWR0107" H 3150 4500 50  0001 C CNN
 F 1 "+5V" H 3150 4790 50  0000 C CNN
 F 2 "" H 3150 4650 50  0001 C CNN
@@
 	2500 5350 2500 6500
 $Comp
-L Device:R R?
+L Device:R R24
 U 1 1 60842AC0
 P 2300 6650
-F 0 "R?" H 2300 6800 50  0000 L CNN
+F 0 "R24" H 2300 6800 50  0000 L CNN
 F 1 "5.1K" V 2300 6550 50  0000 L CNN
 F 2 "Resistor_SMD:R_0603_1608Metric" V 2230 6650 50  0001 C CNN
@@
 $EndComp
 $Comp
-L Device:R R?
+L Device:R R25
 U 1 1 6084514E
 P 2500 6650
-F 0 "R?" H 2500 6800 50  0000 L CNN
+F 0 "R25" H 2500 6800 50  0000 L CNN
 F 1 "5.1K" V 2500 6550 50  0000 L CNN
 F 2 "Resistor_SMD:R_0603_1608Metric" V 2430 6650 50  0001 C CNN
@@
 $EndComp
 $Comp
-L power:GND #PWR?
+L power:GND #PWR0108
 U 1 1 60845610
 P 2400 7000
-F 0 "#PWR?" H 2400 6750 50  0001 C CNN
+F 0 "#PWR0108" H 2400 6750 50  0001 C CNN
 F 1 "GND" H 2405 6827 50  0000 C CNN
 F 2 "" H 2400 7000 50  0001 C CNN
@@
 	4300 4200 4300 4300
 $Comp
-L Device:C C?
+L Device:C C16
 U 1 1 609A562E
 P 3500 6650
-F 0 "C?" H 3550 6750 50  0000 L CNN
+F 0 "C16" H 3550 6750 50  0000 L CNN
 F 1 "47uF" H 3550 6550 50  0000 L CNN
 F 2 "Capacitor_SMD:C_1206_3216Metric" H 3538 6500 50  0001 C CNN
