File: KiCAD/ESP-Hiro/ESP-Hiro.sch (KiCad schematic (older format))
At the start: 70 parts, among them J1 Conn_Q1, J2 Conn_Q2, J3 Conn_Q3, J4 Conn_Q4, J5 Conn_Q5, J6 Conn_ADC, J7 Korean Hroparts TYPE-C-31-M-12, Q1 AO3400A, Q2 AO3400A, Q3 AO3400A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

Commit message: Switch to different USB-C terminal, add some 3d Files, create some better footprints
Parts:
- J1, J2, J3, J4, J5: footprint Connector_Phoenix_MSTB:PhoenixContact_MSTBA_2,5_2-G-5,08_1x02_P5.08mm_Horizontal -> MeineBib:Cixi_Kefa_Elec_KF2EDGR-5.08-2P
- J7: value Korean Hroparts TYPE-C-31-M-12 -> XUNPU TYPEC-304S-ACP16; footprint Connector_USB:USB_C_Receptacle_HRO_TYPE-C-31-M-12 -> MeineBib:USB_C_Receptacle_XUNPU_TYPEC-304S-ACP16; LCSC C165948 -> C720630
Other:
- moved on the sheet: LOGO1
Changed lines of the file:
@@
 L Mechanical:MountingHole LOGO1
 U 1 1 600638EF
-P 1700 -850
-F 0 "LOGO1" H 1800 -804 50  0000 L CNN
-F 1 "Binary-6" H 1800 -895 50  0000 L CNN
-F 2 "MeineBib:Binary_6_v0.1" H 1700 -850 50  0001 C CNN
-F 3 "~" H 1700 -850 50  0001 C CNN
-	1    1700 -850
+P 10950 9100
+F 0 "LOGO1" H 11050 9146 50  0000 L CNN
+F 1 "Binary-6" H 11050 9055 50  0000 L CNN
+F 2 "MeineBib:Binary_6_v0.1" H 10950 9100 50  0001 C CNN
+F 3 "~" H 10950 9100 50  0001 C CNN
+	1    10950 9100
 	1    0    0    -1
 $EndComp
@@
 F 0 "J2" H 15528 3026 50  0000 L CNN
 F 1 "Conn_Q2" H 15250 2900 50  0000 L CNN
-F 2 "Connector_Phoenix_MSTB:PhoenixContact_MSTBA_2,5_2-G-5,08_1x02_P5.08mm_Horizontal" H 15500 3050 50  0001 C CNN
+F 2 "MeineBib:Cixi_Kefa_Elec_KF2EDGR-5.08-2P" H 15500 3050 50  0001 C CNN
 F 3 "~" H 15500 3050 50  0001 C CNN
 F 4 "C8383" H 15500 3050 50  0001 C CNN "LCSC"
@@
 F 0 "J1" H 15528 1476 50  0000 L CNN
 F 1 "Conn_Q1" H 15250 1350 50  0000 L CNN
-F 2 "Connector_Phoenix_MSTB:PhoenixContact_MSTBA_2,5_2-G-5,08_1x02_P5.08mm_Horizontal" H 15500 1500 50  0001 C CNN
+F 2 "MeineBib:Cixi_Kefa_Elec_KF2EDGR-5.08-2P" H 15500 1500 50  0001 C CNN
 F 3 "~" H 15500 1500 50  0001 C CNN
 F 4 "C8383" H 15500 1500 50  0001 C CNN "LCSC"
@@
 F 0 "J3" H 15528 4576 50  0000 L CNN
 F 1 "Conn_Q3" H 15250 4450 50  0000 L CNN
-F 2 "Connector_Phoenix_MSTB:PhoenixContact_MSTBA_2,5_2-G-5,08_1x02_P5.08mm_Horizontal" H 15500 4600 50  0001 C CNN
+F 2 "MeineBib:Cixi_Kefa_Elec_KF2EDGR-5.08-2P" H 15500 4600 50  0001 C CNN
 F 3 "~" H 15500 4600 50  0001 C CNN
 F 4 "C8383" H 15500 4600 50  0001 C CNN "LCSC"
@@
 F 0 "J4" H 15528 6126 50  0000 L CNN
 F 1 "Conn_Q4" H 15250 6000 50  0000 L CNN
-F 2 "Connector_Phoenix_MSTB:PhoenixContact_MSTBA_2,5_2-G-5,08_1x02_P5.08mm_Horizontal" H 15500 6150 50  0001 C CNN
+F 2 "MeineBib:Cixi_Kefa_Elec_KF2EDGR-5.08-2P" H 15500 6150 50  0001 C CNN
 F 3 "~" H 15500 6150 50  0001 C CNN
 F 4 "C8383" H 15500 6150 50  0001 C CNN "LCSC"
@@
 F 0 "J5" H 15528 7676 50  0000 L CNN
 F 1 "Conn_Q5" H 15250 7550 50  0000 L CNN
-F 2 "Connector_Phoenix_MSTB:PhoenixContact_MSTBA_2,5_2-G-5,08_1x02_P5.08mm_Horizontal" H 15500 7700 50  0001 C CNN
+F 2 "MeineBib:Cixi_Kefa_Elec_KF2EDGR-5.08-2P" H 15500 7700 50  0001 C CNN
 F 3 "~" H 15500 7700 50  0001 C CNN
 F 4 "C8383" H 15500 7700 50  0001 C CNN "LCSC"
@@
 P 1500 5750
 F 0 "J7" H 1500 6500 50  0000 C CNN
-F 1 "Korean Hroparts TYPE-C-31-M-12" V 1000 5750 50  0000 C CNN
-F 2 "Connector_USB:USB_C_Receptacle_HRO_TYPE-C-31-M-12" H 1650 5750 50  0001 C CNN
-F 3 "https://datasheet.lcsc.com/szlcsc/1811131825_Korean-Hroparts-Elec-TYPE-C-31-M-12_C165948.pdf" H 1650 5750 50  0001 C CNN
-F 4 "C165948" H 1500 5750 50  0001 C CNN "LCSC"
+F 1 "XUNPU TYPEC-304S-ACP16 " V 1000 5750 50  0000 C CNN
+F 2 "MeineBib:USB_C_Receptacle_XUNPU_TYPEC-304S-ACP16" H 1650 5750 50  0001 C CNN
+F 3 "https://datasheet.lcsc.com/szlcsc/2008152133_XUNPU-TYPEC-304S-ACP16_C720630.pdf" H 1650 5750 50  0001 C CNN
+F 4 "C720630" H 1500 5750 50  0001 C CNN "LCSC"
 	1    1500 5750
 	1    0    0    -1

Commit message: idk
Parts:
- C16: value 47uF -> 10uF; LCSC C96123 -> C13585
Changed lines of the file:
@@
 P 3500 6650
 F 0 "C16" H 3550 6750 50  0000 L CNN
-F 1 "47uF" H 3550 6550 50  0000 L CNN
+F 1 "10uF" H 3550 6550 50  0000 L CNN
 F 2 "Capacitor_SMD:C_1206_3216Metric" H 3538 6500 50  0001 C CNN
 F 3 "~" H 3500 6650 50  0001 C CNN
-F 4 "C96123" H 3500 6650 50  0001 C CNN "LCSC"
+F 4 "C13585" H 3500 6650 50  0001 C CNN "LCSC"
 	1    3500 6650
 	1    0    0    -1
