File: KiCAD/USB-CP2102-only/USB-CP2102-only.sch (KiCad schematic (older format))
At the start: 33 parts, among them J1 5V, J10 TXD, J11 ESP_RST, J12 ESP_GPIO0, J2 V_USB, J3 3.3V, J4 GND, J5 GND, J6 GND, J7 XUNPU TYPEC-304S-ACP16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

Commit message: Wire up initial version of PCB
Parts:
- LOGO1: footprint MeineBib:Binary_6_v0.1 -> MeineBib:LOGO
Changed lines of the file:
@@
 F 0 "LOGO1" H 5350 7396 50  0000 L CNN
 F 1 "Binary-6" H 5350 7305 50  0000 L CNN
-F 2 "MeineBib:Binary_6_v0.1" H 5250 7350 50  0001 C CNN
+F 2 "MeineBib:LOGO" H 5250 7350 50  0001 C CNN
 F 3 "~" H 5250 7350 50  0001 C CNN
 	1    5250 7350
